File: KiCad_Traffic_Light_Controller.kicad_pcb (KiCad board)
At the start: 2 copper layers, 0 parts

Commit message: create pcb design
Parts:
- added C1: 10u, Capacitor_SMD:CP_Elec_4x5.3, F.Cu at (74.5, 94.5)
- added C2: 0.22u, Capacitor_SMD:C_1206_3216Metric_Pad1.33x1.80mm_HandSolder, F.Cu at (142.5, 123.5)
- added C3: 0.22u, Capacitor_SMD:C_1206_3216Metric_Pad1.33x1.80mm_HandSolder, F.Cu at (160.0, 123.5)
- added C4: 100u, Capacitor_SMD:CP_Elec_6.3x5.8, F.Cu at (74.5, 85.0)
- added C5: 0.22u, Capacitor_SMD:C_1206_3216Metric_Pad1.33x1.80mm_HandSolder, F.Cu at (125.5, 123.5)
- added D1: NSC_GRN, LED_THT:LED_D5.0mm, F.Cu at (127.2, 73.8)
- added D10: EWP_RED, LED_THT:LED_D5.0mm, F.Cu at (68.0, 132.2)
- added D11: 1N4148W, Diode_SMD:D_SOD-123, F.Cu at (142.5, 119.5)
- added D12: 1N4148W, Diode_SMD:D_SOD-123, F.Cu at (160.0, 119.5)
- added D13: 1N4148W, Diode_SMD:D_SOD-123, F.Cu at (125.5, 119.0)
- added D2: NSC_YLW, LED_THT:LED_D5.0mm, F.Cu at (127.2, 84.2)
- added D3: NSC_RED, LED_THT:LED_D5.0mm, F.Cu at (127.2, 94.8)
- added D4: EWC_GRN, LED_THT:LED_D5.0mm, F.Cu at (100.3, 116.0)
- added D5: EWC_YLW, LED_THT:LED_D5.0mm, F.Cu at (100.3, 126.0)
- added D6: EWC_RED, LED_THT:LED_D5.0mm, F.Cu at (100.3, 136.0)
- added D7: NSP_GRN, LED_THT:LED_D5.0mm, F.Cu at (160.0, 78.0)
- added D8: NSP_RED, LED_THT:LED_D5.0mm, F.Cu at (160.0, 89.0)
- added D9: EWP_GRN, LED_THT:LED_D5.0mm, F.Cu at (68.0, 122.2)
- added G***: LOGO, logo:ae20, F.Cu at (160.5, 138.0)
- added H1: MountingHole, MountingHole:MountingHole_2.2mm_M2, F.Cu at (58.0, 64.5)
- added H2: MountingHole, MountingHole:MountingHole_2.2mm_M2, F.Cu at (170.5, 64.5)
- added H3: MountingHole, MountingHole:MountingHole_2.2mm_M2, F.Cu at (170.5, 145.0)
- added H4: MountingHole, MountingHole:MountingHole_2.2mm_M2, F.Cu at (58.0, 145.0)
- added J1: Conn_02x08_Odd_Even, Connector_PinHeader_2.54mm:PinHeader_2x08_P2.54mm_Vertical, F.Cu at (88.6, 89.3)
- added J2: Conn_02x08_Odd_Even, Connector_PinHeader_2.54mm:PinHeader_2x08_P2.54mm_Vertical, F.Cu at (88.6, 101.3)
- added J3: Conn_02x05_Odd_Even, Connector_PinHeader_2.54mm:PinHeader_2x05_P2.54mm_Vertical, F.Cu at (95.9, 77.0)
- added J4: +5V, my_footprints:Terminal_Block_5mm, F.Cu at (66.5, 73.0)
- added R1: 130R, Resistor_SMD:R_1206_3216Metric_Pad1.30x1.75mm_HandSolder, F.Cu at (144.5, 70.5)
- added R10: 130R, Resistor_SMD:R_1206_3216Metric_Pad1.30x1.75mm_HandSolder, F.Cu at (91.0, 112.5)
- added R11: 130R, Resistor_SMD:R_1206_3216Metric_Pad1.30x1.75mm_HandSolder, F.Cu at (85.5, 140.5)
- added R12: 130R, Resistor_SMD:R_1206_3216Metric_Pad1.30x1.75mm_HandSolder, F.Cu at (81.5, 140.5)
- added R13: 130R, Resistor_SMD:R_1206_3216Metric_Pad1.30x1.75mm_HandSolder, F.Cu at (77.5, 140.5)
- added R14: 130R, Resistor_SMD:R_1206_3216Metric_Pad1.30x1.75mm_HandSolder, F.Cu at (82.0, 112.5)
- added R15: 130R, Resistor_SMD:R_1206_3216Metric_Pad1.30x1.75mm_HandSolder, F.Cu at (77.5, 112.5)
- added R16: 130R, Resistor_SMD:R_1206_3216Metric_Pad1.30x1.75mm_HandSolder, F.Cu at (89.5, 140.5)
- added R17: 130R, Resistor_SMD:R_1206_3216Metric_Pad1.30x1.75mm_HandSolder, F.Cu at (120.0, 74.0)
- added R18: 130R, Resistor_SMD:R_1206_3216Metric_Pad1.30x1.75mm_HandSolder, F.Cu at (120.0, 84.5)
- added R19: 130R, Resistor_SMD:R_1206_3216Metric_Pad1.30x1.75mm_HandSolder, F.Cu at (120.0, 94.5)
- added R2: 130R, Resistor_SMD:R_1206_3216Metric_Pad1.30x1.75mm_HandSolder, F.Cu at (148.5, 70.5)
- added R20: 130R, Resistor_SMD:R_1206_3216Metric_Pad1.30x1.75mm_HandSolder, F.Cu at (107.5, 116.0)
- added R21: 130R, Resistor_SMD:R_1206_3216Metric_Pad1.30x1.75mm_HandSolder, F.Cu at (107.5, 126.0)
- added R22: 130R, Resistor_SMD:R_1206_3216Metric_Pad1.30x1.75mm_HandSolder, F.Cu at (107.5, 136.0)
- added R23: 130R, Resistor_SMD:R_1206_3216Metric_Pad1.30x1.75mm_HandSolder, F.Cu at (167.0, 78.2)
- added R24: 130R, Resistor_SMD:R_1206_3216Metric_Pad1.30x1.75mm_HandSolder, F.Cu at (167.0, 89.2)
- added R25: 130R, Resistor_SMD:R_1206_3216Metric_Pad1.30x1.75mm_HandSolder, F.Cu at (62.0, 122.0)
- added R26: 130R, Resistor_SMD:R_1206_3216Metric_Pad1.30x1.75mm_HandSolder, F.Cu at (62.0, 132.0)
- added R27: 47K, Resistor_SMD:R_1206_3216Metric_Pad1.30x1.75mm_HandSolder, F.Cu at (160.0, 111.5)
- added R28: 47K, Resistor_SMD:R_1206_3216Metric_Pad1.30x1.75mm_HandSolder, F.Cu at (142.5, 115.5)
- added R29: 47K, Resistor_SMD:R_1206_3216Metric_Pad1.30x1.75mm_HandSolder, F.Cu at (160.0, 115.5)
- added R3: 130R, Resistor_SMD:R_1206_3216Metric_Pad1.30x1.75mm_HandSolder, F.Cu at (144.0, 98.5)
- added R30: 47K, Resistor_SMD:R_1206_3216Metric_Pad1.30x1.75mm_HandSolder, F.Cu at (142.5, 111.5)
- added R31: 47K, Resistor_SMD:R_1206_3216Metric_Pad1.30x1.75mm_HandSolder, F.Cu at (125.5, 115.0)
- added R32: 47K, Resistor_SMD:R_1206_3216Metric_Pad1.30x1.75mm_HandSolder, F.Cu at (125.5, 111.0)
- added R4: 130R, Resistor_SMD:R_1206_3216Metric_Pad1.30x1.75mm_HandSolder, F.Cu at (140.0, 98.5)
- added R5: 130R, Resistor_SMD:R_1206_3216Metric_Pad1.30x1.75mm_HandSolder, F.Cu at (136.0, 98.5)
- added R6: 130R, Resistor_SMD:R_1206_3216Metric_Pad1.30x1.75mm_HandSolder, F.Cu at (140.5, 70.5)
- added R7: 130R, Resistor_SMD:R_1206_3216Metric_Pad1.30x1.75mm_HandSolder, F.Cu at (136.5, 70.5)
- added R8: 130R, Resistor_SMD:R_1206_3216Metric_Pad1.30x1.75mm_HandSolder, F.Cu at (148.0, 98.5)
- added R9: 130R, Resistor_SMD:R_1206_3216Metric_Pad1.30x1.75mm_HandSolder, F.Cu at (86.5, 112.5)
- added SW1: RST, my_footprints:tact_switch_5mm, F.Cu at (152.5, 120.5)
- added SW2: OVR, my_footprints:slide_switch_2.54mm, F.Cu at (135.5, 117.5)
- added SW3: EN, my_footprints:slide_switch_2.54mm, F.Cu at (119.0, 117.5)
- added U1: SM420561N, Display_7Segment:7SegmentLED_LTS6760_LTS6780, F.Cu at (137.4, 92.1)
- added U2: SM420561N, Display_7Segment:7SegmentLED_LTS6760_LTS6780, F.Cu at (78.4, 134.1)
- added U3: LM1117DT-3.3, Package_TO_SOT_SMD:SOT-223, F.Cu at (64.5, 88.5)
Routing:
- net GND: track 0.00 -> 448.4 mm, vias 0 -> 4
- net /+3.3V: track 0.00 -> 263.4 mm, vias 0 -> 4
- net /EN: track 0.00 -> 142.7 mm
- net /RST: track 0.00 -> 134.9 mm, vias 0 -> 2
- net /OVR: track 0.00 -> 122.9 mm, vias 0 -> 2
- net /NS_HEX_A: track 0.00 -> 104.0 mm
- net /NS_HEX_B: track 0.00 -> 91.8 mm
- net /+5V: track 0.00 -> 83.8 mm
- net /EW_HEX_D: track 0.00 -> 76.2 mm
- net /EW_HEX_C: track 0.00 -> 71.6 mm
- net /NSP_GRN: track 0.00 -> 68.2 mm
- net /NSP_RED: track 0.00 -> 67.7 mm
- net /EW_HEX_E: track 0.00 -> 67.4 mm, vias 0 -> 1
- net /EW_HEX_DP: track 0.00 -> 64.9 mm, vias 0 -> 1
- net /NSC_GRN: track 0.00 -> 60.9 mm, vias 0 -> 2
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Other:
- board outline added: 121.5 x 89.5 mm
- board text added: "+3.3V"
- board text added: "+5V"
- board text added: "A"
- board text added: "B"
- board text added: "C"
- board text added: "CAR"
- board text added: "Control Logic Connector"
- board text added: "D"
- board text added: "DP"
- board text added: "E"
- board text added: "E-W"
- board text added: "EAST-WEST TRAFFIC LIGHTS"
- board text added: "EN"
- board text added: "ENABLE"
- board text added: "EW Connector"
- board text added: "F"
- board text added: "G"
- board text added: "GABRIEL G. OROZCO 21 APRIL 2026 Computer Engineering Technology Department Technological University of the Philippines Visayas"
- board text added: "GND"
- board text added: "N-S"
- board text added: "NORTH-SOUTH TRAFFIC LIGHTS"
- board text added: "NS Connector"
- board text added: "OVERRIDE"
- board text added: "OVR"
- board text added: "PED"
- board text added: "R"
- board text added: "RESET"
- board text added: "RST"
- board text added: "Traffic Light Controller board for Finite State Machine (FSM) demo. It manages traffic flow for two perpendicular roads: North-South (NS) and East-West (EW)."
- board text added: "Y"
